Commit message: - Fixed controller.yaml - Fixed inertia

File: robot_test1_description/urdf/base/base.urdf.xacro (robot description, xacro)
@@ -24,5 +24,5 @@
       </collision>
       <inertial>
-        <origin xyz="0 0 0" rpy="0 0 0"/>
+        <origin xyz="${offset} 0 0" rpy="0 0 0"/>
         <mass value="${mass}"/>
         <inertia

File: robot_test1_description/urdf/wheel/idler_wheel.urdf.xacro (robot description, xacro)
@@ -26,5 +26,5 @@
       </collision>
       <inertial>
-        <origin xyz="0 0 0" rpy="0 0 0"/>
+        <origin xyz="0 0 -${z_offset/2}" rpy="0 0 0"/>
         <mass value="${mass}"/>
         <inertia
